Commit message: pk added

File: src/darwin_description/urdf/darwin.urdf (robot description, URDF)
Before this commit: robot darwinOP, 31 links, 30 joints
Links:
- link MP_ANKLE1_L: geometry collision mesh filename=../meshes/ankle1_l_coll.stl scale=1 1 1; visual mesh filename=../meshes/ankle1_l.STL scale=1 1 1
- link MP_ANKLE1_R: geometry collision mesh filename=../meshes/ankle1_r_coll.stl scale=1 1 1; visual mesh filename=../meshes/ankle1_r.STL scale=1 1 1
- link MP_ANKLE2_L: geometry collision mesh filename=../meshes/ankle2_l_coll.stl scale=1 1 1; visual mesh filename=../meshes/ankle2_l.STL scale=1 1 1
- link MP_ANKLE2_R: geometry collision mesh filename=../meshes/ankle2_r_coll.stl scale=1 1 1; visual mesh filename=../meshes/ankle2_r.STL scale=1 1 1
- link MP_ARM_HIGH_L: geometry collision mesh filename=../meshes/arm_high_l_coll.stl scale=1 1 1; visual mesh filename=../meshes/arm_high_l.STL scale=1 1 1
- link MP_ARM_HIGH_R: geometry collision mesh filename=../meshes/arm_high_r_coll.stl scale=1 1 1; visual mesh filename=../meshes/arm_high_r.STL scale=1 1 1
- link MP_BODY: geometry collision mesh filename=../meshes/body_coll.stl scale=1 1 1; visual mesh filename=../meshes/body.STL scale=1 1 1
- link MP_HEAD: geometry collision mesh filename=../meshes/head_coll.stl scale=1 1 1; visual mesh filename=../meshes/head.STL scale=1 1 1
- link MP_NECK: geometry collision mesh filename=../meshes/neck_coll.stl scale=1 1 1; visual mesh filename=../meshes/neck.STL scale=1 1 1
- link MP_PELVIS_L: geometry collision mesh filename=../meshes/pelvis_l_coll.stl scale=1 1 1; visual mesh filename=../meshes/pelvis_l.STL scale=1 1 1
- link MP_PELVIS_R: geometry collision mesh filename=../meshes/pelvis_r_coll.stl scale=1 1 1; visual mesh filename=../meshes/pelvis_r.STL scale=1 1 1
- link MP_SHOULDER_L: geometry collision mesh filename=../meshes/shoulder_l_coll.stl scale=1 1 1; visual mesh filename=../meshes/shoulder_l.STL scale=1 1 1
- link MP_SHOULDER_R: geometry collision mesh filename=../meshes/shoulder_r_coll.stl scale=1 1 1; visual mesh filename=../meshes/shoulder_r.STL scale=1 1 1
- link MP_THIGH1_L: geometry collision mesh filename=../meshes/thigh1_l_coll.stl scale=1 1 1; visual mesh filename=../meshes/thigh1_l.STL scale=1 1 1
- link MP_THIGH1_R: geometry collision mesh filename=../meshes/thigh1_r_coll.stl scale=1 1 1; visual mesh filename=../meshes/thigh1_r.STL scale=1 1 1
- link MP_THIGH2_L: geometry collision mesh filename=../meshes/thigh2_l_coll.stl scale=1 1 1; visual mesh filename=../meshes/thigh2_l.STL scale=1 1 1
- link MP_THIGH2_R: geometry collision mesh filename=../meshes/thigh2_r_coll.stl scale=1 1 1; visual mesh filename=../meshes/thigh2_r.STL scale=1 1 1
- link MP_TIBIA_L: geometry collision mesh filename=../meshes/tibia_l_coll.stl scale=1 1 1; visual mesh filename=../meshes/tibia_l.STL scale=1 1 1
- link MP_TIBIA_R: geometry collision mesh filename=../meshes/tibia_r_coll.stl scale=1 1 1; visual mesh filename=../meshes/tibia_r.STL scale=1 1 1
